Commit message: works MPCWBC in gazebo simulator with feetplacement constraint

File: catkin_ws/src/Jueying_description/X20/urdf/X20_model.xacro (robot description, xacro)
@@ -519,4 +519,31 @@
   </joint>
     <!-- ros_control plugin -->
+  <gazebo reference="BASE">
+    <material>Gazebo/Blue</material>
+  </gazebo>
+  <gazebo reference="RH_SHANK">
+    <material>Gazebo/Orange</material>
+  </gazebo>
+  <gazebo reference="LH_SHANK">
+    <material>Gazebo/Orange</material>
+  </gazebo>
+  <gazebo reference="RF_SHANK">
+    <material>Gazebo/Orange</material>
+  </gazebo>
+  <gazebo reference="LF_SHANK">
+    <material>Gazebo/Orange</material>
+  </gazebo>
+  <gazebo reference="RH_THIGH">
+    <material>Gazebo/Green</material>
+  </gazebo>
+  <gazebo reference="LH_THIGH">
+    <material>Gazebo/Green</material>
+  </gazebo>
+  <gazebo reference="RF_THIGH">
+    <material>Gazebo/Green</material>
+  </gazebo>
+  <gazebo reference="LF_THIGH">
+    <material>Gazebo/Green</material>
+  </gazebo>
   <gazebo>
     <plugin name="gazebo_ros_control" filename="libgazebo_ros_control.so">

Commit message: x20 gazebo sim, local trajectory(velocity interface)

File: catkin_ws/src/Jueying_description/X20/urdf/X20_model.xacro (robot description, xacro)
@@ -65,5 +65,5 @@
     <child link="imu_link"/>
   </joint>
-  <link name="velodyne">
+  <!-- <link name="velodyne">
     <inertial>
       <mass value="0.0000001"/>
@@ -89,5 +89,9 @@
     <parent link="BASE"/>
     <child link="velodyne"/>
-  </joint>
+  </joint> -->
+ <xacro:include filename="$(find velodyne_description)/urdf/HDL-32E.urdf.xacro"/>
+  <xacro:HDL-32E parent="BASE" name="velodyne2" topic="/velodyne_points_32"  hz="10" samples="220" >
+    <origin xyz="0.35 0 0.6" rpy="0 0.5 0" />
+  </xacro:HDL-32E>
     <link name="camera_link">
     <inertial>
@@ -114,5 +118,5 @@
   <joint name="camera_to_velodyne" type="fixed">
     <origin xyz="0.013274 -0.035092 0.0245" rpy="0 0 0" />
-    <parent link="velodyne" />
+    <parent link="velodyne2" />
     <child link="camera_link" />
     <axis xyz="0 0 1" />
@@ -610,5 +614,5 @@
   </gazebo>
   <!-- Gazebo requires the velodyne_gazebo_plugins package -->
-  <gazebo reference="velodyne">
+  <!-- <gazebo reference="velodyne">
     <sensor name="velodyne-VLP16" type="ray">
       <pose>0 0 0 0 0 0</pose>
@@ -649,5 +653,5 @@
       </plugin>
     </sensor>
-  </gazebo>
+  </gazebo> -->
   <!-- Joint 'implicitSpringDamper' setup, according to official website's suggestion-->
   <xacro:macro name="joint_setup_block" params="joint_name">

Commit message: change the swingplanner eventime, copy the previous swing trajectories according to the current event time.

File: catkin_ws/src/Jueying_description/X20/urdf/X20_model.xacro (robot description, xacro)
@@ -92,5 +92,5 @@
  <xacro:include filename="$(find velodyne_description)/urdf/HDL-32E.urdf.xacro"/>
   <xacro:HDL-32E parent="BASE" name="velodyne2" topic="/velodyne_points_32"  hz="10" samples="220" >
-    <origin xyz="0.35 0 0.6" rpy="0 0.5 0" />
+    <origin xyz="0.35 0 0.5" rpy="0 0.4 0" />
   </xacro:HDL-32E>
     <link name="camera_link">

Commit message: camera on robot & topic same

File: catkin_ws/src/Jueying_description/X20/urdf/X20_model.xacro (robot description, xacro)
@@ -3,13 +3,4 @@
   <xacro:property name="motor_damp" value="1.2"/>
   <xacro:property name="motor_fric" value="0.1"/>
-  <!-- <link name="origin_link">
-    </link>
-  <joint name="origin_joint" type="fixed">
-    <origin
-      xyz="0 0 1"
-      rpy="0 0 0"/>
-    <parent link="origin_link"/>
-    <child link="BASE"/>
-  </joint> -->
   <link
     name="BASE">
@@ -65,61 +56,20 @@
     <child link="imu_link"/>
   </joint>
-  <!-- <link name="velodyne">
-    <inertial>
-      <mass value="0.0000001"/>
-      <origin rpy="0 0 0" xyz="0 0 0"/>
-      <inertia ixx="0.0000000001" ixy="0" ixz="0" iyy="0.00000000001" iyz="0" izz="0.000000001"/>
-    </inertial>
-  <visual>
-    <origin rpy="0 0 0" xyz="0 0 0"/>
-    <geometry>
-      <box size="0.01 0.01 0.01"/>
-    </geometry>
-  </visual>
-  <collision>
-    <origin rpy="0 0 0" xyz="0 0 0"/>
-    <geometry>
-      <box size=".001 .001 .001"/>
-    </geometry>
-  </collision>
- </link>
- <joint name="velodyne_joint" type="fixed">
-    <axis xyz="0 0 0"/>
-    <origin xyz="0.4 0 0.2"/>
-    <parent link="BASE"/>
-    <child link="velodyne"/>
-  </joint> -->
  <xacro:include filename="$(find velodyne_description)/urdf/HDL-32E.urdf.xacro"/>
-  <xacro:HDL-32E parent="BASE" name="velodyne2" topic="/velodyne_points_32"  hz="10" samples="220" >
+  <xacro:HDL-32E parent="BASE" name="lidar_link" topic="/point_cloud2"  hz="10" samples="220" >
     <origin xyz="0.35 0 0.5" rpy="0 0.4 0" />
   </xacro:HDL-32E>
-    <link name="camera_link">
-    <inertial>
-      <mass value="0.0000001"/>
-      <origin rpy="0 0 0" xyz="0 0 0"/>
-      <inertia ixx="0.0000000001" ixy="0" ixz="0" iyy="0.00000000001" iyz="0" izz="0.000000001"/>
-    </inertial>
-    <visual>
-      <origin  xyz="0 0 0"  rpy="0 0 0" />
-      <geometry>
-        <mesh filename="package://X20/meshes/camera_Link.STL" />
-      </geometry>
-      <material name="">
-        <color rgba="0.250980392156863 0.250980392156863 0.250980392156863 1" />
-      </material>
-    </visual>
-    <collision>
-      <origin xyz="0 0 0" rpy="0 0 0" />
-      <geometry>
-        <mesh filename="package://X20/meshes/camera_Link.STL" />
-      </geometry>
-    </collision>
-  </link>
-  <joint name="camera_to_velodyne" type="fixed">
-    <origin xyz="0.013274 -0.035092 0.0245" rpy="0 0 0" />
-    <parent link="velodyne2" />
-    <child link="camera_link" />
-    <axis xyz="0 0 1" />
-  </joint>
+  <xacro:include filename="$(find X20)/urdf/kinect.xacro"/>
+  <xacro:property name="M_PI" value="3.14159" />
+  <xacro:kinect_camera prefix="camera"/>
+  <joint name="kinect_frame_joint" type="fixed">
+    <origin xyz="0.35 0 0.3" rpy="0 0.3 0" />
+    <parent link="BASE"/>
+    <child link="camera_link"/>
+  </joint>
+  <!-- <xacro:include filename="$(find realsense_ros_gazebo)/xacro/depthcam.xacro"/>
+  <xacro:realsense_d435 sensor_name="d435" parent_link="BASE" rate="10">
+    <origin rpy="0 0 0.5 " xyz="0.1 0 0.45"/>
+  </xacro:realsense_d435> -->
   <link name="LF_HIP">
     <inertial>

Commit message: mhz gazebo

File: catkin_ws/src/Jueying_description/X20/urdf/X20_model.xacro (robot description, xacro)
@@ -64,5 +64,5 @@
   <xacro:kinect_camera prefix="camera"/>
   <joint name="kinect_frame_joint" type="fixed">
-    <origin xyz="0.35 0 0.3" rpy="0 0.3 0" />
+    <origin xyz="0.7 0 1" rpy="0 1.3 0" />
     <parent link="BASE"/>
     <child link="camera_link"/>

Commit message: camera pose

File: catkin_ws/src/Jueying_description/X20/urdf/X20_model.xacro (robot description, xacro)
@@ -64,5 +64,5 @@
   <xacro:kinect_camera prefix="camera"/>
   <joint name="kinect_frame_joint" type="fixed">
-    <origin xyz="0.7 0 1" rpy="0 1.3 0" />
+    <origin xyz="0.3 0 -0.08" rpy="0 1.4 0" />
     <parent link="BASE"/>
     <child link="camera_link"/>

Commit message: sim test in 2023/07/02 14:32pm mhz

File: catkin_ws/src/Jueying_description/X20/urdf/X20_model.xacro (robot description, xacro)
@@ -92,5 +92,5 @@
  <xacro:include filename="$(find velodyne_description)/urdf/HDL-32E.urdf.xacro"/>
   <xacro:HDL-32E parent="BASE" name="velodyne2" topic="/velodyne_points_32"  hz="10" samples="220" >
-    <origin xyz="0.35 0 0.5" rpy="0 0.4 0" />
+    <origin xyz="0.4 0 0.5" rpy="0 0.8 0" />
   </xacro:HDL-32E>
     <link name="camera_link">
