Commit message: before Qutintic spline

File: ocs2_ws/src/jy_control_gazebo/legged_x20_description/urdf/X20_model.xacro (robot description, xacro)
@@ -94,5 +94,5 @@
     <origin xyz="0.35 0 0.6" rpy="0 0.5 0" />
   </xacro:HDL-32E>
-    <link name="camerlink">
+    <!-- <link name="camerlink">
     <inertial>
       <mass value="0.0000001"/>
@@ -121,5 +121,5 @@
     <child link="camerlink" />
     <axis xyz="0 0 1" />
-  </joint>
+  </joint> -->
   <link name="LF_HIP">
     <inertial>

Commit message: ros control 2023/07/02 sim test in 104 after meeting.

File: ocs2_ws/src/jy_control_gazebo/legged_x20_description/urdf/X20_model.xacro (robot description, xacro)
@@ -514,5 +514,5 @@
     <child link = "RH_FOOT"/>
   </joint>
-  <xacro:property name="foot_mass" value="0.06"/>
+  <xacro:property name="foot_mass" value="0.001"/>
   <xacro:property name="foot_radius" value="0.036"/>
   <xacro:macro name="setup_foot" params="link_name">

Commit message: sim in deep 2023/07/04 plan to merge to mip.

File: ocs2_ws/src/jy_control_gazebo/legged_x20_description/urdf/X20_model.xacro (robot description, xacro)
@@ -92,5 +92,5 @@
  <xacro:include filename="$(find velodyne_description)/urdf/HDL-32E.urdf.xacro"/>
   <xacro:HDL-32E parent="BASE" name="lidar_link" topic="/point_cloud2"  hz="10" samples="220" >
-    <origin xyz="0.35 0 0.6" rpy="0 0.5 0" />
+    <origin xyz="0.45 0 0.8" rpy="0 1 0" />
   </xacro:HDL-32E>
     <!-- <link name="camerlink">

Commit message: world

File: ocs2_ws/src/jy_control_gazebo/legged_x20_description/urdf/X20_model.xacro (robot description, xacro)
@@ -92,5 +92,5 @@
  <xacro:include filename="$(find velodyne_description)/urdf/HDL-32E.urdf.xacro"/>
   <xacro:HDL-32E parent="BASE" name="lidar_link" topic="/point_cloud2"  hz="10" samples="220" >
-    <origin xyz="0.35 0 0.6" rpy="0 0.5 0" />
+    <origin xyz="0.35 0 0.5" rpy="0 0.9 0" />
   </xacro:HDL-32E>
     <!-- <link name="camerlink">

Commit message: add mhz niuqu world,urdf lidar position change, tf close

File: ocs2_ws/src/jy_control_gazebo/legged_x20_description/urdf/X20_model.xacro (robot description, xacro)
@@ -92,5 +92,5 @@
  <xacro:include filename="$(find velodyne_description)/urdf/HDL-32E.urdf.xacro"/>
   <xacro:HDL-32E parent="BASE" name="lidar_link" topic="/point_cloud2"  hz="10" samples="220" >
-    <origin xyz="0.35 0 0.5" rpy="0 0.9 0" />
+    <origin xyz="0.7 0 0.4" rpy="0 1 0" />
   </xacro:HDL-32E>
     <!-- <link name="camerlink">

File: ocs2_ws/src/jy_control_gazebo/legged_x20_description/urdf/gazebo_x20/X20_gazebo.xacro (robot description, xacro)
@@ -7,4 +7,4 @@
   <xacro:include filename="$(find legged_x20_description)/urdf/gazebo_x20/imu.xacro"/>
   <xacro:IMU connected_to="BASE" imu_name="unitree_imu" xyz="0. 0. 0." rpy="0. 0. 0."/>
-  <xacro:include filename="$(find legged_x20_description)/urdf/gazebo_x20/gazebo.xacro"/>s
+  <xacro:include filename="$(find legged_x20_description)/urdf/gazebo_x20/gazebo.xacro"/>
 </robot>

Commit message: A LARGE STEP

File: ocs2_ws/src/jy_control_gazebo/legged_x20_description/urdf/X20_model.xacro (robot description, xacro)
@@ -19,5 +19,5 @@
         rpy="0 0 0" />
       <mass
-        value="26.398" />
+        value="26.398" />  <!-- 29.398 -->
       <inertia ixx="0.1632" ixy="-5.2136E-05" ixz="-0.00019406" iyy="0.40648" iyz="8.2679E-05" izz="0.52596" />
     </inertial>
@@ -92,5 +92,5 @@
  <xacro:include filename="$(find velodyne_description)/urdf/HDL-32E.urdf.xacro"/>
   <xacro:HDL-32E parent="BASE" name="lidar_link" topic="/point_cloud2"  hz="10" samples="220" >
-    <origin xyz="0.7 0 0.4" rpy="0 1 0" />
+    <origin xyz="0.4 0 0.8" rpy="0 1.05 0" />
   </xacro:HDL-32E>
     <!-- <link name="camerlink">

Commit message: FIXME: Foot trajectory not turned off, unable to walk blindly

File: ocs2_ws/src/jy_control_gazebo/legged_x20_description/urdf/X20_model.xacro (robot description, xacro)
@@ -1,6 +1,6 @@
 <?xml version="1.0" encoding="utf-8"?>
 <robot name="X20" xmlns:xacro="http://www.ros.org/wiki/xacro">
-  <xacro:property name="motor_damp" value="1.2"/>
-  <xacro:property name="motor_fric" value="0.1"/>
+  <xacro:property name="motor_damp" value="1.2" />
+  <xacro:property name="motor_fric" value="0.1" />
   <!-- <link name="origin_link">
     </link>
@@ -20,5 +20,6 @@
       <mass
         value="26.398" />
-      <inertia ixx="0.1632" ixy="-5.2136E-05" ixz="-0.00019406" iyy="0.40648" iyz="8.2679E-05" izz="0.52596" />
+      <inertia ixx="0.1632" ixy="-5.2136E-05" ixz="-0.00019406" iyy="0.40648" iyz="8.2679E-05"
+        izz="0.52596" />
     </inertial>
     <visual>
@@ -42,26 +43,26 @@
   <link name="imu_link">
     <inertial>
-      <mass value="0.0000001"/>
-      <origin rpy="0 0 0" xyz="0 0 0"/>
-      <inertia ixx="0.0000000001" ixy="0" ixz="0" iyy="0.00000000001" iyz="0" izz="0.000000001"/>
-    </inertial>
-  <visual>
-    <origin rpy="0 0 0" xyz="0 0 0"/>
-    <geometry>
-      <box size="0.001 0.001 0.001"/>
-    </geometry>
-  </visual>
-  <collision>
-    <origin rpy="0 0 0" xyz="0 0 0"/>
-    <geometry>
-      <box size=".001 .001 .001"/>
-    </geometry>
-  </collision>
- </link>
- <joint name="imu_joint" type="fixed">
-    <axis xyz="0 0 0"/>
-    <origin xyz="0 0 0"/>
-    <parent link="BASE"/>
-    <child link="imu_link"/>
+      <mass value="0.0000001" />
+      <origin rpy="0 0 0" xyz="0 0 0" />
+      <inertia ixx="0.0000000001" ixy="0" ixz="0" iyy="0.00000000001" iyz="0" izz="0.000000001" />
+    </inertial>
+    <visual>
+      <origin rpy="0 0 0" xyz="0 0 0" />
+      <geometry>
+        <box size="0.001 0.001 0.001" />
+      </geometry>
+    </visual>
+    <collision>
+      <origin rpy="0 0 0" xyz="0 0 0" />
+      <geometry>
+        <box size=".001 .001 .001" />
+      </geometry>
+    </collision>
+  </link>
+  <joint name="imu_joint" type="fixed">
+    <axis xyz="0 0 0" />
+    <origin xyz="0 0 0" />
+    <parent link="BASE" />
+    <child link="imu_link" />
   </joint>
   <!-- <link name="velodyne">
@@ -90,9 +91,10 @@
     <child link="velodyne"/>
   </joint> -->
- <xacro:include filename="$(find velodyne_description)/urdf/HDL-32E.urdf.xacro"/>
-  <xacro:HDL-32E parent="BASE" name="lidar_link" topic="/point_cloud2"  hz="10" samples="220" >
-    <origin xyz="0.7 0 0.4" rpy="0 1 0" />
+  <xacro:include filename="$(find velodyne_description)/urdf/HDL-32E.urdf.xacro" />
+  <xacro:HDL-32E parent="BASE" name="lidar_link" topic="/point_cloud2" hz="10" samples="220">
+    <origin xyz="0.5 0 0.6" rpy="0 0.4 0" />
+    <!-- <origin xyz="0.7 0 0.4" rpy="0 1 0" /> -->
   </xacro:HDL-32E>
-    <!-- <link name="camerlink">
+  <!-- <link name="camerlink">
     <inertial>
       <mass value="0.0000001"/>
@@ -126,5 +128,6 @@
       <origin xyz="-0.00075689 -0.0089129 -5.0528E-05" />
       <mass value="1.5767" />
-      <inertia ixx="0.0012141" ixy="6.1989E-06" ixz="2.8652E-06" iyy="0.0016912" iyz="3.7E-06" izz="0.0013431" />
+      <inertia ixx="0.0012141" ixy="6.1989E-06" ixz="2.8652E-06" iyy="0.0016912" iyz="3.7E-06"
+        izz="0.0013431" />
     </inertial>
     <visual>
@@ -148,5 +151,5 @@
       upper="0.38397"
       effort="126.1"
-      velocity="12"  />
+      velocity="12" />
     <dynamics
       damping="${motor_damp}"
@@ -157,5 +160,6 @@
       <origin xyz="-0.0025264 -0.022118 -0.0292" />
       <mass value="3.0063" />
-      <inertia ixx="0.0058102" ixy="4.2848E-05" ixz="-3.0437E-06" iyy="0.0080686" iyz="-6.889E-05" izz="0.003874" />
+      <inertia ixx="0.0058102" ixy="4.2848E-05" ixz="-3.0437E-06" iyy="0.0080686" iyz="-6.889E-05"
+        izz="0.003874" />
     </inertial>
     <visual>
@@ -179,5 +183,5 @@
       upper="0.48869"
       effort="111.4"
-      velocity="19"/>
+      velocity="19" />
     <dynamics
       damping="${motor_damp}"
@@ -210,5 +214,5 @@
       upper="2.84488"
       effort="195.8"
-      velocity="19"  />
+      velocity="19" />
     <dynamics
       damping="${motor_damp}"
@@ -241,5 +245,5 @@
       upper="0.38397"
       effort="126.1"
-      velocity="12"  />
+      velocity="12" />
     <dynamics
       damping="${motor_damp}"
@@ -250,5 +254,6 @@
       <origin xyz="-0.0025264 -0.022118 -0.0292" />
       <mass value="3.0063" />
-      <inertia ixx="0.0058102" ixy="4.2848E-05" ixz="-3.0433E-06" iyy="0.008" iyz="-6.8889E-05" izz="0.003874" />
+      <inertia ixx="0.0058102" ixy="4.2848E-05" ixz="-3.0433E-06" iyy="0.008" iyz="-6.8889E-05"
+        izz="0.003874" />
     </inertial>
     <visual>
@@ -272,5 +277,5 @@
       upper="0.48869"
       effort="111.4"
-      velocity="19"/>
+      velocity="19" />
     <dynamics
       damping="${motor_damp}"
@@ -303,5 +308,5 @@
       upper="2.84488"
       effort="195.8"
-      velocity="19"  />
+      velocity="19" />
     <dynamics
       damping="${motor_damp}"
@@ -312,5 +317,6 @@
       <origin xyz="-0.000757 0.009 5.0528E-05" />
       <mass value="1.5767" />
-      <inertia ixx="0.0012141" ixy="-6.1989E-06" ixz="-2.8652E-06" iyy="0.0016912" iyz="3.7E-06" izz="0.0013431" />
+      <inertia ixx="0.0012141" ixy="-6.1989E-06" ixz="-2.8652E-06" iyy="0.0016912" iyz="3.7E-06"
+        izz="0.0013431" />
     </inertial>
     <visual>
@@ -334,5 +340,5 @@
       upper="0.38397"
       effort="126.1"
-      velocity="12"  />
+      velocity="12" />
     <dynamics
       damping="${motor_damp}"
@@ -343,5 +349,6 @@
       <origin xyz="-0.0025266 0.022119 -0.029194" />
       <mass value="3.0062" />
-      <inertia ixx="0.00581" ixy="-4.2781E-05" ixz="-3.0682E-06" iyy="0.0080684" iyz="6.8812E-05" izz="0.0038739" />
+      <inertia ixx="0.00581" ixy="-4.2781E-05" ixz="-3.0682E-06" iyy="0.0080684" iyz="6.8812E-05"
+        izz="0.0038739" />
     </inertial>
     <visual>
@@ -365,5 +372,5 @@
       upper="0.48869"
       effort="111.4"
-      velocity="19"/>
+      velocity="19" />
     <dynamics
       damping="${motor_damp}"
@@ -396,5 +403,5 @@
       upper="2.84488"
       effort="195.8"
-      velocity="19"  />
+      velocity="19" />
     <dynamics
       damping="${motor_damp}"
@@ -405,5 +412,6 @@
       <origin xyz="0.00075689 0.0089129 -5.0528E-05" />
       <mass value="1.5767" />
-      <inertia ixx="0.0012141" ixy="6.1989E-06" ixz="-2.8652E-06" iyy="0.0016912" iyz="-3.7E-06" izz="0.0013431" />
+      <inertia ixx="0.0012141" ixy="6.1989E-06" ixz="-2.8652E-06" iyy="0.0016912" iyz="-3.7E-06"
+        izz="0.0013431" />
     </inertial>
     <visual>
@@ -427,5 +435,5 @@
       upper="0.38397"
       effort="126.1"
-      velocity="12"  />
+      velocity="12" />
     <dynamics
       damping="${motor_damp}"
@@ -436,5 +444,6 @@
       <origin xyz="-0.0025266 0.022119 -0.029194" />
       <mass value="3.0062" />
-      <inertia ixx="0.00581" ixy="-4.2781E-05" ixz="-3.0681E-06" iyy="0.0080684" iyz="6.8812E-05" izz="0.0038739" />
+      <inertia ixx="0.00581" ixy="-4.2781E-05" ixz="-3.0681E-06" iyy="0.0080684" iyz="6.8812E-05"
+        izz="0.0038739" />
     </inertial>
     <visual>
@@ -458,5 +467,5 @@
       upper="0.48869"
       effort="111.4"
-      velocity="19"/>
+      velocity="19" />
     <dynamics
       damping="${motor_damp}"
@@ -467,5 +476,6 @@
       <origin xyz="0.0075224 2.589E-05 -0.17586" />
       <mass value="0.54849" />
-      <inertia ixx="0.0056981" ixy="1.1608E-07" ixz="0.00015292" iyy="0.0059026" iyz="-1.1243E-06" izz="0.00028822" />
+      <inertia ixx="0.0056981" ixy="1.1608E-07" ixz="0.00015292" iyy="0.0059026" iyz="-1.1243E-06"
+        izz="0.00028822" />
     </inertial>
     <visual>
@@ -489,53 +499,53 @@
       upper="2.84488"
       effort="195.8"
-      velocity="19"  />
-    <dynamics
-      damping="${motor_damp}"
-      friction="${motor_fric}" />
-  </joint>
-  <joint name = "LF_FOOT_joint" type = "fixed">
-    <origin xyz="0 0 -0.33" rpy = "0 0 0"/>
-    <parent link="LF_SHANK"/>
-    <child link = "LF_FOOT"/>
-  </joint>
-  <joint name = "LH_FOOT_joint" type = "fixed">
-    <origin xyz="0 0 -0.33" rpy = "0 0 0"/>
-    <parent link="LH_SHANK"/>
-    <child link = "LH_FOOT"/>
-  </joint>
-  <joint name = "RF_FOOT_joint" type = "fixed">
-    <origin xyz="0 0 -0.33" rpy = "0 0 0"/>
-    <parent link="RF_SHANK"/>
-    <child link = "RF_FOOT"/>
-  </joint>
-  <joint name = "RH_FOOT_joint" type = "fixed">
-    <origin xyz="0 0 -0.33" rpy = "0 0 0"/>
-    <parent link="RH_SHANK"/>
-    <child link = "RH_FOOT"/>
-  </joint>
-  <xacro:property name="foot_mass" value="0.001"/>
-  <xacro:property name="foot_radius" value="0.036"/>
+      velocity="19" />
+    <dynamics
+      damping="${motor_damp}"
+      friction="${motor_fric}" />
+  </joint>
+  <joint name="LF_FOOT_joint" type="fixed">
+    <origin xyz="0 0 -0.33" rpy="0 0 0" />
+    <parent link="LF_SHANK" />
+    <child link="LF_FOOT" />
+  </joint>
+  <joint name="LH_FOOT_joint" type="fixed">
+    <origin xyz="0 0 -0.33" rpy="0 0 0" />
+    <parent link="LH_SHANK" />
+    <child link="LH_FOOT" />
+  </joint>
+  <joint name="RF_FOOT_joint" type="fixed">
+    <origin xyz="0 0 -0.33" rpy="0 0 0" />
+    <parent link="RF_SHANK" />
+    <child link="RF_FOOT" />
+  </joint>
+  <joint name="RH_FOOT_joint" type="fixed">
+    <origin xyz="0 0 -0.33" rpy="0 0 0" />
+    <parent link="RH_SHANK" />
+    <child link="RH_FOOT" />
+  </joint>
+  <xacro:property name="foot_mass" value="0.001" />
+  <xacro:property name="foot_radius" value="0.036" />
   <xacro:macro name="setup_foot" params="link_name">
     <link name="${link_name}">
-        <visual>
-            <origin rpy="0 0 0" xyz="0 0 0"/>
-            <geometry>
-                <sphere radius="${foot_radius-0.01}"/>
-            </geometry>
-            <material name="orange"/>
-        </visual>
-        <collision>
-            <origin rpy="0 0 0" xyz="0 0 0"/>
-            <geometry>
-                <sphere radius="${foot_radius}"/>
-            </geometry>
-        </collision>
-        <inertial>
-            <mass value="${foot_mass}"/>
-            <inertia
-                    ixx="${(2*foot_mass)/5.0*(foot_radius*foot_radius)}" ixy="0.0" ixz="0.0"
-                    iyy="${(2*foot_mass)/5.0*(foot_radius*foot_radius)}" iyz="0.0"
-                    izz="${(2*foot_mass)/5.0*(foot_radius*foot_radius)}"/>
-        </inertial>
+      <visual>
+        <origin rpy="0 0 0" xyz="0 0 0" />
+        <geometry>
+          <sphere radius="${foot_radius-0.01}" />
+        </geometry>
+        <material name="orange" />
+      </visual>
+      <collision>
+        <origin rpy="0 0 0" xyz="0 0 0" />
+        <geometry>
+          <sphere radius="${foot_radius}" />
+        </geometry>
+      </collision>
+      <inertial>
+        <mass value="${foot_mass}" />
+        <inertia
+          ixx="${(2*foot_mass)/5.0*(foot_radius*foot_radius)}" ixy="0.0" ixz="0.0"
+          iyy="${(2*foot_mass)/5.0*(foot_radius*foot_radius)}" iyz="0.0"
+          izz="${(2*foot_mass)/5.0*(foot_radius*foot_radius)}" />
+      </inertial>
     </link>
     <gazebo reference="${link_name}_joint">
@@ -543,17 +553,17 @@
     </gazebo>
     <gazebo reference="${link_name}">
-        <mu1>0.8</mu1>
-        <mu2>0.8</mu2>
-        <self_collide>1</self_collide>
-        <material>Gazebo/DarkGrey</material>
-        <kp value="1000000.0"/>
-        <kd value="100.0"/>
+      <mu1>0.8</mu1>
+      <mu2>0.8</mu2>
+      <self_collide>1</self_collide>
+      <material>Gazebo/DarkGrey</material>
+      <kp value="1000000.0" />
+      <kd value="100.0" />
     </gazebo>
   </xacro:macro>
-  <xacro:setup_foot link_name="LF_FOOT"/>
-  <xacro:setup_foot link_name="LH_FOOT"/>
-  <xacro:setup_foot link_name="RF_FOOT"/>
-  <xacro:setup_foot link_name="RH_FOOT"/>
-    <!-- ros_control plugin -->
+  <xacro:setup_foot link_name="LF_FOOT" />
+  <xacro:setup_foot link_name="LH_FOOT" />
+  <xacro:setup_foot link_name="RF_FOOT" />
+  <xacro:setup_foot link_name="RH_FOOT" />
+  <!-- ros_control plugin -->
   <gazebo reference="BASE">
     <material>Gazebo/Blue</material>
@@ -609,5 +619,5 @@
     </sensor>
   </gazebo> -->
-<!-- <gazebo reference="camerlink">
+  <!-- <gazebo reference="camerlink">
     <sensor type="camera" name="camernode">
       <update_rate>15.0</update_rate>
@@ -712,12 +722,12 @@
       <self_collide>1</self_collide>
       <material>Gazebo/DarkGrey</material>
-      <kp value="1000000.0"/>
-      <kd value="100.0"/>
+      <kp value="1000000.0" />
+      <kd value="100.0" />
     </gazebo>
   </xacro:macro>
-  <xacro:link_setup_block link_name="LF_SHANK"/>
-  <xacro:link_setup_block link_name="LH_SHANK"/>
-  <xacro:link_setup_block link_name="RF_SHANK"/>
-  <xacro:link_setup_block link_name="RH_SHANK"/>
+  <xacro:link_setup_block link_name="LF_SHANK" />
+  <xacro:link_setup_block link_name="LH_SHANK" />
+  <xacro:link_setup_block link_name="RF_SHANK" />
+  <xacro:link_setup_block link_name="RH_SHANK" />
   <xacro:macro name="link_setup_block_hip" params="link_name">
     <gazebo reference="${link_name}">
@@ -733,15 +743,15 @@
       <self_collide>0</self_collide>
       <material>Gazebo/DarkGrey</material>
-      <kp value="1000000.0"/>
-      <kd value="100.0"/>
+      <kp value="1000000.0" />
+      <kd value="100.0" />
     </gazebo>
   </xacro:macro>
-  <xacro:link_setup_block_hip link_name="LF_HIP"/>
-  <xacro:link_setup_block_thight link_name="LF_THIGH"/>
-  <xacro:link_setup_block_hip link_name="RF_HIP"/>
-  <xacro:link_setup_block_thight link_name="RF_THIGH"/>
-  <xacro:link_setup_block_hip link_name="LH_HIP"/>
-  <xacro:link_setup_block_thight link_name="LH_THIGH"/>
-  <xacro:link_setup_block_hip link_name="RH_HIP"/>
-  <xacro:link_setup_block_thight link_name="RH_THIGH"/>
+  <xacro:link_setup_block_hip link_name="LF_HIP" />
+  <xacro:link_setup_block_thight link_name="LF_THIGH" />
+  <xacro:link_setup_block_hip link_name="RF_HIP" />
+  <xacro:link_setup_block_thight link_name="RF_THIGH" />
+  <xacro:link_setup_block_hip link_name="LH_HIP" />
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
Commit message: ocs2_wbc & ocs2_wbc_ros & ocs2_raisim for legged_footholds.

File: ocs2_ws/src/jy_control_gazebo/legged_x20_description/urdf/X20_model.xacro (robot description, xacro)
@@ -93,4 +93,5 @@
   <xacro:HDL-32E parent="BASE" name="lidar_link" topic="/point_cloud2"  hz="10" samples="220" >
     <origin xyz="0.4 0 0.8" rpy="0 1.05 0" />
+    <!-- <origin xyz="0.4 0 0.1" rpy="0 0 0" /> -->
   </xacro:HDL-32E>
     <!-- <link name="camerlink">
