Commit message: real X20 test in 2022/11/01 add base mass to X20_rsm.urdf and add z weight

File: ocs2_ws/src/X20/urdf/X20_rsm.urdf (robot description, URDF)
Before this commit: robot X20, 18 links, 17 joints
Links:
- link INERTIA: mass 26.398 -> 32.398

Commit message: ready to merge NewMpcWbcinSDK

File: ocs2_ws/src/X20/urdf/X20_rsm.urdf (robot description, URDF)
Before this commit: robot X20, 18 links, 17 joints
Links:
- added link lidar_link; visual mesh filename=package://X20/meshes/velodyne.STL
- link LF_SHANK: geometry collision sphere radius=0.05; visual mesh filename=package://X20/meshes/Shank.dae
- link LH_SHANK: geometry collision sphere radius=0.05; visual mesh filename=package://X20/meshes/Shank.dae
- link RF_SHANK: geometry collision sphere radius=0.05; visual mesh filename=package://X20/meshes/Shank.dae
- link RH_SHANK: geometry collision sphere radius=0.05; visual mesh filename=package://X20/meshes/Shank.dae
Joints:
- added joint lidar_joint: type fixed, parent base, child lidar_link, origin xyz=0.25 0 0.309 rpy=0 0.4 0

Commit message: disable feedback mpc to avoid large gain of control input. add some param in launch

File: ocs2_ws/src/X20/urdf/X20_rsm.urdf (robot description, URDF)
Before this commit: robot X20, 19 links, 18 joints
Links:
- link LF_SHANK: geometry collision cylinder length=0.32 radius=0.02; collision sphere radius=0.02
- link LH_SHANK: geometry collision cylinder length=0.32 radius=0.02; collision sphere radius=0.02
- link RF_SHANK: geometry collision cylinder length=0.32 radius=0.02; collision sphere radius=0.02
- link RH_SHANK: geometry collision cylinder length=0.32 radius=0.02; collision sphere radius=0.02

Commit message: change frame name 'base' to 'BASE' in X20_rsm.urdf, 2023/06/27 17:00 sim test with ZR in deep Robotics.

File: ocs2_ws/src/X20/urdf/X20_rsm.urdf (robot description, URDF)
Before this commit: robot X20, 19 links, 18 joints
Links:
- removed link base
- added link BASE; collision box size=0.46 0.26 0.15; visual mesh filename=package://X20/meshes/Torso.dae
Joints:
- joint Base2Inertia: parent base -> BASE
- joint LF_HAA: parent base -> BASE
- joint LH_HAA: parent base -> BASE
- joint RF_HAA: parent base -> BASE
- joint RH_HAA: parent base -> BASE
- joint lidar_joint: parent base -> BASE

Commit message: After IROS 2024 [0326]

File: ocs2_ws/src/X20/urdf/X20_rsm.urdf (robot description, URDF)
Before this commit: robot X20, 19 links, 18 joints
Links:
- removed link lidar_link
- link LF_SHANK: geometry collision cylinder length=0.32 radius=0.02; collision sphere radius=0.036
- link LH_SHANK: geometry collision cylinder length=0.32 radius=0.02; collision sphere radius=0.036
- link RF_SHANK: geometry collision cylinder length=0.32 radius=0.02; collision sphere radius=0.036
- link RH_SHANK: geometry collision cylinder length=0.32 radius=0.02; collision sphere radius=0.036
Joints:
- removed joint lidar_joint

Commit message: NB: ready to real dog, Lu Chen' advice, raisim scanThread.

File: ocs2_ws/src/X20/urdf/X20_rsm.urdf (robot description, URDF)
Before this commit: robot X20, 18 links, 17 joints
Links:
- added link lidar_link; visual mesh filename=package://X20/meshes/velodyne.STL
Joints:
- added joint lidar_joint: type fixed, parent BASE, child lidar_link, origin xyz=0.25 0 0.309 rpy=0 0.4 0

Commit message: elevation_close_loop

File: ocs2_ws/src/X20/urdf/X20_rsm.urdf (robot description, URDF)
Before this commit: robot X20, 19 links, 18 joints
Joints:
- joint lidar_joint: origin xyz=0.25 0 0.309 rpy=0 0.4 0 -> xyz=0.13 0 0.2 rpy=0 0.0 0

Commit message: elevation_close_loop reed shepp planning

File: ocs2_ws/src/X20/urdf/X20_rsm.urdf (robot description, URDF)
Before this commit: robot X20, 19 links, 18 joints
Links:
- removed link BASE
- added link base; collision box size=0.46 0.26 0.15; visual mesh filename=package://X20/meshes/Torso.dae
Joints:
- joint Base2Inertia: parent BASE -> base
- joint LF_HAA: parent BASE -> base
- joint LH_HAA: parent BASE -> base
- joint RF_HAA: parent BASE -> base
- joint RH_HAA: parent BASE -> base
- joint lidar_joint: parent BASE -> base

Commit message: add pronto-base est in sim, fix some zyx and xyz eular bugs in global planner. MPC_WBC_sim rm catkin_ws, X20_rsm add imu sensor

File: ocs2_ws/src/X20/urdf/X20_rsm.urdf (robot description, URDF)
Before this commit: robot X20, 19 links, 18 joints
Links:
- added link imu_link
Joints:
- added joint base_to_imu: type fixed, parent base, child imu_link, origin xyz=0.0 0.0 0.0 rpy=0.0 0.0 0.0
